Commit message: updates

File: pointfoot-legged-gym/resources/robots/PF_TRON1A/urdf/robot_with_basket_processed.urdf (robot description, URDF)
Before this commit: robot point_foot_tron1a_with_basket, 14 links, 13 joints
Joints:
- joint base_to_contact_plate: origin xyz=0 0 0.15 rpy=0 0 0 -> xyz=0 0 0.02 rpy=0 0 0
